File: design/piaa/power.kicad_sch (KiCad schematic)
At the start: 14 parts, among them J8 Screw_Terminal_01x02, U10 NCP1117-3.3_SOT223, U9 LM2596S-5

Commit message: update to pcb drawing
Parts:
- J8: footprint Connector_PinHeader_2.00mm:PinHeader_1x02_P2.00mm_Horizontal -> Connector_PinHeader_2.00mm:PinHeader_1x02_P2.00mm_Vertical
Changed lines of the file:
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@@
     (property "Reference" "J8" (id 0) (at 72.39 87.63 0))
     (property "Value" "Screw_Terminal_01x02" (id 1) (at 66.04 95.25 0))
-    (property "Footprint" "Connector_PinHeader_2.00mm:PinHeader_1x02_P2.00mm_Horizontal" (id 2) (at 72.39 90.17 0)
+    (property "Footprint" "Connector_PinHeader_2.00mm:PinHeader_1x02_P2.00mm_Vertical" (id 2) (at 72.39 90.17 0)
       (effects (font (size 1.27 1.27)) hide)
     )

Commit message: updates to schematic
Other:
- company: (none) -> Patricio Whittingslow
- title: (none) -> PIAA (power)
Changed lines of the file:
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@@
 (kicad_sch (version 20211123) (generator eeschema)
   (paper "A4")
+  (title_block
+    (title "PIAA (power)")
+    (date "t March 2023")
+    (rev "A.0")
+    (company "Patricio Whittingslow")
+  )
   (junction (at 113.03 90.17) (diameter 0) (color 0 0 0 0)
   )

Commit message: fix header and bornier size
Parts:
- J8: footprint Connector_PinHeader_2.00mm:PinHeader_1x02_P2.00mm_Vertical -> TerminalBlock:TerminalBlock_bornier-2_P5.08mm
Changed lines of the file:
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@@
     (property "Reference" "J8" (id 0) (at 72.39 87.63 0))
     (property "Value" "Screw_Terminal_01x02" (id 1) (at 66.04 95.25 0))
-    (property "Footprint" "Connector_PinHeader_2.00mm:PinHeader_1x02_P2.00mm_Vertical" (id 2) (at 72.39 90.17 0)
+    (property "Footprint" "TerminalBlock:TerminalBlock_bornier-2_P5.08mm" (id 2) (at 72.39 90.17 0)
       (effects (font (size 1.27 1.27)) hide)
     )
